Commit message: O carro aparece agora

File: wenis_ws/install/arm_pkg/share/arm_pkg/urdf/manipulator.xacro (robot description, xacro)
@@ -22,5 +22,5 @@
     </link>
     <joint name="manipulator_fixed" type="fixed">
-        <origin xyz="0 0 0.0025" rpy="0 0 0"/>
+        <origin xyz="0 0 0.3025" rpy="0 0 0"/>
         <parent link="world"/>
         <child link="base_0"/>

File: wenis_ws/install/platform/share/platform/urdf/platform.xacro (robot description, xacro)
@@ -4,8 +4,15 @@
 	<!-- This is the body of the robot -->
 	<link name="body_link">
+	    <inertial>
+		    <mass value="5"/>
+			<origin xyz="0 0 0.15"/>
+			<inertia ixx="0.02216" ixy="5.8001e-06" ixz="6.1941e-06" iyy="0.024835"
+					iyz="-5.3034e-05"
+					izz="0.021063"/>
+		</inertial>
 		<visual>
 			<origin rpy="0 0 0" xyz="0 0 0.15"/>
 			<geometry>
-				<box size="1 0.6 0.3" />
+				<box size="1 0.6 0.3"/>
 			</geometry>
 			<material name="red">
@@ -13,17 +20,30 @@
 			</material>
 		</visual>
+        <collision>
+	        <origin rpy="0 0 0" xyz="0 0 0.15"/>
+            <geometry>
+                <box size="1 0.6 0.3"/>
+            </geometry>
+        </collision>
 	</link>
 	<!-- This is the back right wheel of the robot -->
-	<joint name="wheel1_joint" type="continuous" >
+	<joint name="wheel1_joint" type="continuous">
 		<parent link="body_link"/>
-		<child link="wheel1_link" />
-		<origin xyz="-0.3 -0.35 -0.1" rpy="0 0 0" />
-		<axis xyz="0 1 0" />
+		<child link="wheel1_link"/>
+		<origin xyz="-0.3 -0.35 -0.1" rpy="0 0 0"/>
+		<axis xyz="0 1 0"/>
 	</joint>
 	<link name="wheel1_link">
+	    <inertial>
+		    <mass value="1.5"/>
+			<origin xyz="-0.3 -0.35 -0.1"/>
+			<inertia ixx="0.02216" ixy="5.8001e-06" ixz="6.1941e-06" iyy="0.024835"
+					iyz="-5.3034e-05"
+					izz="0.021063"/>
+		</inertial>
 		<visual>
-			<origin rpy="1.570795 0 0" xyz="0 0 0" />
+			<origin rpy="1.570795 0 0" xyz="0 0 0"/>
 			<geometry>
-				<cylinder length="0.1" radius="0.15" />
+				<cylinder length="0.1" radius="0.15"/>
 			</geometry>
 			<material name="yellow">
@@ -31,17 +51,30 @@
 			</material>
 		</visual>
+        <collision>
+	        <origin rpy="1.570795 0 0" xyz="0 0 0"/>
+            <geometry>
+                <cylinder length="0.1" radius="0.15"/>
+            </geometry>
+        </collision>
 	</link>
 	<!-- This is the back left wheel of the robot -->
-	<joint name="wheel2_joint" type="continuous" >
+	<joint name="wheel2_joint" type="continuous">
 		<parent link="body_link"/>
-		<child link="wheel2_link" />
-		<origin xyz="-0.3 0.35 -0.1" rpy="0 0 0" />
-		<axis xyz="0 1 0" />
+		<child link="wheel2_link"/>
+		<origin xyz="-0.3 0.35 -0.1" rpy="0 0 0"/>
+		<axis xyz="0 1 0"/>
 	</joint>
 	<link name="wheel2_link">
+	    <inertial>
+		    <mass value="1.5"/>
+			<origin xyz="-0.3 0.35 -0.1"/>
+			<inertia ixx="0.02216" ixy="5.8001e-06" ixz="6.1941e-06" iyy="0.024835"
+					iyz="-5.3034e-05"
+					izz="0.021063"/>
+		</inertial>
 		<visual>
-			<origin rpy="1.570795 0 0" xyz="0 0 0" />
+			<origin rpy="1.570795 0 0" xyz="0 0 0"/>
 			<geometry>
-				<cylinder length="0.1" radius="0.15" />
+				<cylinder length="0.1" radius="0.15"/>
 			</geometry>
 			<material name="yellow">
@@ -49,17 +82,30 @@
 			</material>
 		</visual>
+        <collision>
+            <origin rpy="1.570795 0 0" xyz="0 0 0"/>
+            <geometry>
+                <cylinder length="0.1" radius="0.15"/>
+            </geometry>
+        </collision>
 	</link>
 	<!-- This is the front right wheel of the robot -->
-	<joint name="wheel3_joint" type="continuous" >
+	<joint name="wheel3_joint" type="continuous">
 		<parent link="body_link"/>
-		<child link="wheel3_link" />
-		<origin xyz="0.3 -0.35 -0.1" rpy="0 0 0" />
-		<axis xyz="0 1 0" />
+		<child link="wheel3_link"/>
+		<origin xyz="0.3 -0.35 -0.1" rpy="0 0 0"/>
+		<axis xyz="0 1 0"/>
 	</joint>
 	<link name="wheel3_link">
+	    <inertial>
+		    <mass value="1.5"/>
+			<origin xyz="0.3 -0.35 -0.1"/>
+			<inertia ixx="0.02216" ixy="5.8001e-06" ixz="6.1941e-06" iyy="0.024835"
+					iyz="-5.3034e-05"
+					izz="0.021063"/>
+		</inertial>
 		<visual>
-			<origin rpy="1.570795 0 0" xyz="0 0 0" />
+			<origin rpy="1.570795 0 0" xyz="0 0 0"/>
 			<geometry>
-				<cylinder length="0.1" radius="0.15" />
+				<cylinder length="0.1" radius="0.15"/>
 			</geometry>
 			<material name="yellow">
@@ -67,17 +113,30 @@
 			</material>
 		</visual>
+        <collision>
+		    <origin rpy="1.570795 0 0" xyz="0 0 0"/>
+            <geometry>
+                <cylinder length="0.1" radius="0.15"/>
+            </geometry>
+        </collision>
 	</link>
 	<!-- This is the front left wheel of the robot -->
-	<joint name="wheel4_joint" type="continuous" >
+	<joint name="wheel4_joint" type="continuous">
 		<parent link="body_link"/>
-		<child link="wheel4_link" />
-		<origin xyz="0.3 0.35 -0.1" rpy="0 0 0" />
-		<axis xyz="0 1 0" />
+		<child link="wheel4_link"/>
+		<origin xyz="0.3 0.35 -0.1" rpy="0 0 0"/>
+		<axis xyz="0 1 0"/>
 	</joint>
 	<link name="wheel4_link">
+	    <inertial>
+		    <mass value="1.5"/>
+			<origin xyz="0.3 0.35 -0.1"/>
+			<inertia ixx="0.02216" ixy="5.8001e-06" ixz="6.1941e-06" iyy="0.024835"
+					iyz="-5.3034e-05"
+					izz="0.021063"/>
+		</inertial>
 		<visual>
-			<origin rpy="1.570795 0 0" xyz="0 0 0" />
+			<origin rpy="1.570795 0 0" xyz="0 0 0"/>
 			<geometry>
-				<cylinder length="0.1" radius="0.15" />
+				<cylinder length="0.1" radius="0.15"/>
 			</geometry>
 			<material name="yellow">
@@ -85,4 +144,10 @@
 			</material>
 		</visual>
+        <collision>
+		    <origin rpy="1.570795 0 0" xyz="0 0 0"/>
+            <geometry>
+                <cylinder length="0.1" radius="0.15"/>
+            </geometry>
+        </collision>
 	</link>
 </robot>

Commit message: DESESPERO

File: wenis_ws/install/arm_pkg/share/arm_pkg/urdf/manipulator.xacro (robot description, xacro)
@@ -22,5 +22,5 @@
     </link>
     <joint name="manipulator_fixed" type="fixed">
-        <origin xyz="0 0 0.3025" rpy="0 0 0"/>
+        <origin xyz="0 0 0.0025" rpy="0 0 0"/>
         <parent link="world"/>
         <child link="base_0"/>
