Commit message: Boas-vindas das férias
Não sei o que diabos está acontecendo.

File: wenis_ws/install/arm_pkg/share/arm_pkg/urdf/arm_platform.xacro (robot description, xacro)
@@ -2,28 +2,5 @@
 <robot xmlns:xacro="http://ros.org/wiki/xacro" name="robot_description">
     <xacro:include filename="$(find arm_pkg)/urdf/new_a0912.urdf.xacro" />
-    <xacro:include filename="$(find arm_pkg)/urdf/depth_camera.xacro"/>
     <xacro:manipulator namespace=""/>
-    <link name="world">
-    <visual>
-        <origin xyz="0 0 0" rpy="0 0 0"/>
-        <geometry>
-            <box size="5.0 5.0 0.05"/>
-        </geometry>
-        <material name="Grey">
-            <color rgba="0.7 0.7 0.7 1.0"/>
-        </material>
-    </visual>
-    <collision>
-        <origin xyz="0 0 0" rpy="0 0 0"/>
-        <geometry>
-            <box size="5.0 5.0 0.05"/>
-        </geometry>
-    </collision>
-    </link>
-    <joint name="manipulator_fixed" type="fixed">
-        <origin xyz="5 0 0.0025" rpy="0 0 0"/>
-        <parent link="world"/>
-        <child link="base_0"/>
-    </joint>
     <!-- Load Common Material -->
     <xacro:include filename="$(find xarm_description)/urdf/common/common.material.xacro" />

File: wenis_ws/install/arm_pkg/share/arm_pkg/urdf/new_a0912.urdf.xacro (robot description, xacro)
@@ -1,4 +1,4 @@
 <?xml version="1.0"?>
-<robot xmlns:xacro="http://www.ros.org/wiki/xacro" name="a0912" >
+<robot xmlns:xacro="http://www.ros.org/wiki/xacro" name="new_a0912" >
   <xacro:macro name="manipulator" params="namespace">
     <xacro:arg name="color"   default="blue"/>
@@ -7,6 +7,6 @@
     <xacro:property name="cr" value="$(arg color)"/>
     <xacro:property name="gr" value="$(arg gripper)"/>
-     <xacro:include filename="$(find arm_pkg)/urdf/macro.a0912.blue.xacro" />
-     <xacro:a0912 namespace="$(arg namespace)"/>
+     <xacro:include filename="$(find arm_pkg)/urdf/new_macro.a0912.blue.xacro" />
+     <xacro:new_a0912 namespace="$(arg namespace)"/>
   </xacro:macro>
 </robot>

File: wenis_ws/install/arm_pkg/share/arm_pkg/urdf/new_macro.a0912.blue.xacro (robot description, xacro)
@@ -1,9 +1,9 @@
 <?xml version="1.0"?>
-<robot name="a0912" xmlns:xacro="http://www.ros.org/wiki/xacro">
+<robot name="new_a0912" xmlns:xacro="http://www.ros.org/wiki/xacro">
 	<xacro:include filename="$(find arm_pkg)/urdf/macro.gazebo_config_control.xacro" />
 	<xacro:include filename="$(find arm_pkg)/urdf/macro.transmission.xacro" />
 	<xacro:include filename="$(find arm_pkg)/urdf/macro.internal_config.xacro" />
 	<xacro:include filename="$(find arm_pkg)/urdf/macro.bumper_config.xacro" />
-	<xacro:macro name="a0912" params="namespace">
+	<xacro:macro name="new_a0912" params="namespace">
         <link name="body_link">
 	        <inertial>
@@ -158,5 +158,5 @@
 			<inertial>
 				<mass value="3.635"/>
-				<origin xyz="4e-06   -0.001016     0.38181"/>
+				<origin xyz="4e-06   -0.001016     0.53181"/>
 				<inertia ixx="0.02216" ixy="5.8001e-06" ixz="6.1941e-06" iyy="0.024835"
 					iyz="-5.3034e-05"
@@ -164,5 +164,5 @@
 			</inertial>
 			<visual>
-				<origin rpy="0 0 0" xyz="0 0 0.3" />
+				<origin rpy="0 0 0" xyz="0 0 0.45" />
 				<geometry>
 					<mesh filename="file:///$(find arm_pkg)/meshes/a0912_blue/A0912_0_0.dae" scale="0.001 0.001 0.001" />
@@ -178,5 +178,5 @@
 			<parent link="body_link"/>
 			<child link="base_0"/>
-			<origin xyz="0 0 0.3" rpy="0 0 0"/>
+			<origin xyz="0 0 0.45" rpy="0 0 0"/>
 			<axis xyz="0 0 1"/>
 		</joint>
@@ -185,5 +185,5 @@
 			<parent link="base_0" />
 			<child link="link1" />
-			<origin rpy="0 0 0" xyz="0 0 0.495" />
+			<origin rpy="0 0 0" xyz="0 0 0.645" />
 			<axis xyz="0 0 1" />
 			<limit effort="411" lower="-6.2832" upper="6.2832" velocity="3.1416"/>
