Commit message: Agora ele não sai vazado

File: wenis_ws/install/platform/share/platform/urdf/aplatform.xacro (robot description, xacro)
@@ -21,4 +21,11 @@
                 </geometry>
             </collision>
+            <inertial>
+		<mass value="1.5"/>
+	        <origin xyz="0 0 0.15"/>
+		<inertia ixx="0.02216" ixy="5.8001e-06" ixz="6.1941e-06" iyy="0.024835"
+					iyz="-5.3034e-05"
+					izz="0.021063"/>
+	    </inertial>
 	</link>
 	<joint name="manipulator_fixed" type="fixed">
@@ -49,25 +56,25 @@
 	<link name="wheel1_link">
 	    <inertial>
-		    <mass value="1.5"/>
-			<origin xyz="-0.3 -0.35 0"/>
-			<inertia ixx="0.02216" ixy="5.8001e-06" ixz="6.1941e-06" iyy="0.024835"
+		<mass value="1.5"/>
+	        <origin xyz="-0.3 -0.35 0"/>
+		<inertia ixx="0.02216" ixy="5.8001e-06" ixz="6.1941e-06" iyy="0.024835"
 					iyz="-5.3034e-05"
 					izz="0.021063"/>
-		</inertial>
-		<visual>
-			<origin rpy="1.570795 0 0" xyz="0 0 0"/>
-			<geometry>
-				<cylinder length="0.1" radius="0.15"/>
-			</geometry>
-			<material name="yellow">
-				<color rgba="1 1 0 1"/>
-			</material>
-		</visual>
-        <collision>
+	    </inertial>
+	    <visual>
+		<origin rpy="1.570795 0 0" xyz="0 0 0"/>
+		<geometry>
+			<cylinder length="0.1" radius="0.15"/>
+		</geometry>
+		<material name="yellow">
+			<color rgba="1 1 0 1"/>
+		</material>
+	    </visual>
+            <collision>
 	        <origin rpy="1.570795 0 0" xyz="0 0 0"/>
-            <geometry>
-                <cylinder length="0.1" radius="0.15"/>
-            </geometry>
-        </collision>
+                <geometry>
+                        <cylinder length="0.1" radius="0.15"/>
+                </geometry>
+            </collision>
 	</link>
 	<!-- This is the back left wheel of the robot -->

Commit message: Tentativas de ajustes

File: wenis_ws/install/platform/share/platform/urdf/aplatform.xacro (robot description, xacro)
@@ -22,13 +22,13 @@
             </collision>
             <inertial>
-		<mass value="1.5"/>
+		<mass value="6"/>
 	        <origin xyz="0 0 0.15"/>
-		<inertia ixx="0.02216" ixy="5.8001e-06" ixz="6.1941e-06" iyy="0.024835"
+		<inertia ixx="0.22216" ixy="5.8001e-06" ixz="6.1941e-06" iyy="0.224835"
 					iyz="-5.3034e-05"
-					izz="0.021063"/>
+					izz="0.221063"/>
 	    </inertial>
 	</link>
 	<joint name="manipulator_fixed" type="fixed">
-          <origin xyz="0 0 0.3" rpy="0 0 0"/>
+          <origin xyz="-0.021001 0.0002 0.3" rpy="0 0 0"/>
           <parent link="body_link"/>
           <child link="base_0"/>

File: wenis_ws/src/ros2_manipulator/robotic_arm_environment/platform/urdf/aplatform.xacro (robot description, xacro)
@@ -22,13 +22,13 @@
             </collision>
             <inertial>
-		<mass value="5.1"/>
-	        <origin xyz="-0.3 -0.35 0"/>
-		<inertia ixx="0.02216" ixy="5.8001e-06" ixz="6.1941e-06" iyy="0.024835"
+		<mass value="6"/>
+	        <origin xyz="0 0 0.15"/>
+		<inertia ixx="0.22216" ixy="5.8001e-06" ixz="6.1941e-06" iyy="0.224835"
 					iyz="-5.3034e-05"
-					izz="0.021063"/>
+					izz="0.221063"/>
 	    </inertial>
 	</link>
 	<joint name="manipulator_fixed" type="fixed">
-          <origin xyz="0 0 0.3" rpy="0 0 0"/>
+          <origin xyz="-0.021001 0.0002 0.3" rpy="0 0 0"/>
           <parent link="body_link"/>
           <child link="base_0"/>

Commit message: Mudanças na garra

File: wenis_ws/install/platform/share/platform/urdf/aplatform.xacro (robot description, xacro)
@@ -3,4 +3,5 @@
 <robot xmlns:xacro="http://ros.org/wiki/xacro" name="robot_description">
         <xacro:include filename="$(find arm_pkg)/urdf/a0912.urdf.xacro" />
+        <xacro:include filename="$(find robotiq_85_description)/urdf/robotiq_85_gripper_macro_gz.urdf.xacro" />
         <xacro:manipulator namespace=""/>
 	<!-- This is the body of the robot -->
@@ -40,11 +41,7 @@
         <!-- gazebo use -->
         <xacro:property name="mesh_path" value="file://$(find xarm_description)/meshes" />
-        <!-- include the GRIPPER -->
-        <xacro:include filename="$(find xarm_description)/urdf/common/common.link.xacro" />
-        <xacro:parse_link_inertial_filename dof="6" robot_type="xarm" robot_sn="" model1300="false" />
-        <xacro:property name="inertial_params_filename" value="${scope_parent_inertial_params_filename}"/>
-        <xacro:property name="new_model1300" value="${scope_parent_model1300}"/>
-        <xacro:include filename="$(find xarm_description)/urdf/gripper/xarm_gripper_macro.xacro" />
-        <xacro:xarm_gripper_macro prefix="" attach_to="link6" ros2_control_plugin="gazebo_ros2_control/GazeboSystem" dof="6" hard_interface="PositionJointInterface" />
+        <xacro:robotiq_85_gripper prefix="" parent="link6" >
+           <origin xyz="0.0 0 0.0" rpy="0 -1.57 1.57"/>
+        </xacro:robotiq_85_gripper>
 	<!-- This is the back right wheel of the robot -->
 	<joint name="wheel1_joint" type="continuous">
