Commit message: pfc
Add "new_arm_ws"

File: new_arm_ws/install/cr35ia_ros2_gazebo/share/cr35ia_ros2_gazebo/urdf/cr35ia_macro.urdf.xacro (robot description, xacro)
@@ -237,4 +237,5 @@
       <axis xyz="0 0 1"/>
       <limit lower="-2.9670" upper="2.9670" effort="0" velocity="3.1415"/>
+      <dynamics damping="50.0" friction="1.0"/>
     </joint>
     <joint name="${prefix}joint_2" type="revolute">
@@ -244,4 +245,5 @@
       <axis xyz="0 1 0"/>
       <limit lower="-0.7853" upper="2.0943" effort="0" velocity="3.1415"/>
+      <dynamics damping="50.0" friction="1.0"/>
     </joint>
     <joint name="${prefix}joint_3" type="revolute">
@@ -251,4 +253,5 @@
       <axis xyz="0 -1 0"/>
       <limit lower="-2.1450" upper="2.3561" effort="0" velocity="3.4906"/>
+      <dynamics damping="10.0" friction="1.0"/>
     </joint>
     <joint name="${prefix}joint_4" type="revolute">
@@ -258,4 +261,5 @@
       <axis xyz="-1 0 0"/>
       <limit lower="-3.4906" upper="3.4906" effort="0" velocity="6.1086"/>
+      <dynamics damping="5.0" friction="1.0"/>
     </joint>
     <joint name="${prefix}joint_5" type="revolute">
@@ -265,4 +269,5 @@
       <axis xyz="0 -1 0"/>
       <limit lower="-1.9198" upper="1.9198" effort="0" velocity="6.1086"/>
+      <dynamics damping="2.0" friction="1.0"/>
     </joint>
     <joint name="${prefix}joint_6" type="revolute">
@@ -272,4 +277,5 @@
       <axis xyz="-1 0 0"/>
       <limit lower="-7.8539" upper="7.8539" effort="0" velocity="6.9813"/>
+      <dynamics damping="1.0" friction="1.0"/>
     </joint>
     <!-- end of joint list -->

File: new_arm_ws/install/iiwa_ros2_gazebo/share/iiwa_ros2_gazebo/urdf/iiwa_macro.urdf.xacro (robot description, xacro)
@@ -251,4 +251,5 @@
       <axis xyz="0 0 1" />
       <limit lower="-2.9668" upper="2.9668" effort="0" velocity="1.4834" />
+      <dynamics damping="0.5" friction="1.0"/>
     </joint>
     <joint name="${prefix}joint_2" type="revolute">
@@ -258,4 +259,5 @@
       <axis xyz="0 1 0" />
       <limit lower="-2.0942" upper="2.0942" effort="0" velocity="1.4834" />
+      <dynamics damping="0.5" friction="1.0"/>
     </joint>
     <joint name="${prefix}joint_3" type="revolute">
@@ -265,4 +267,5 @@
       <axis xyz="0 0 1" />
       <limit lower="-2.9668" upper="2.9668" effort="0" velocity="1.7452" />
+      <dynamics damping="0.5" friction="1.0"/>
     </joint>
     <joint name="${prefix}joint_4" type="revolute">
@@ -272,4 +275,5 @@
       <axis xyz="0 -1 0" />
       <limit lower="-2.0942" upper="2.0942" effort="0" velocity="1.3089" />
+      <dynamics damping="0.5" friction="1.0"/>
     </joint>
     <joint name="${prefix}joint_5" type="revolute">
@@ -279,4 +283,5 @@
       <axis xyz="0 0 1" />
       <limit lower="-2.9668" upper="2.9668" effort="0" velocity="2.2688" />
+      <dynamics damping="0.5" friction="1.0"/>
     </joint>
     <joint name="${prefix}joint_6" type="revolute">
@@ -286,4 +291,5 @@
       <axis xyz="0 1 0" />
       <limit lower="-2.0942" upper="2.0942" effort="0" velocity="2.356" />
+      <dynamics damping="0.5" friction="1.0"/>
     </joint>
     <joint name="${prefix}joint_7" type="revolute">
@@ -293,4 +299,5 @@
       <axis xyz="0 0 1" />
       <limit lower="-3.0541" upper="3.0541" effort="0" velocity="2.356" />
+      <dynamics damping="0.5" friction="1.0"/>
     </joint>
     <!-- end of joint list -->

File: new_arm_ws/install/irb1200_ros2_gazebo/share/irb1200_ros2_gazebo/urdf/irb1200_macro.urdf.xacro (robot description, xacro)
@@ -21,10 +21,10 @@
 #           Phil Webb        - p.f.webb@cranfield.ac.uk                                 #
 #                                                                                       #
-#  Date: September, 2022.                                                                    #
-#                                                                                       #
-# ===================================== COPYRIGHT ===================================== #
-# ===================================== COPYRIGHT ===================================== #
-#                                                                                       #
-#  Some of the information used to build the ROS2 ABB-IRB1200 .urdf files in this ROS2   #
+#  Date: September, 2022.                                                               #
+#                                                                                       #
+# ===================================== COPYRIGHT ===================================== #
+# ===================================== COPYRIGHT ===================================== #
+#                                                                                       #
+#  Some of the information used to build the ROS2 ABB-IRB1200 .urdf files in this ROS2  #
 #  repository has been taken from the following resource:                               #
 #       - abb_experimental (https://github.com/ros-industrial/abb_experimental)         #

File: new_arm_ws/install/irb1200_ros2_gazebo/share/irb1200_ros2_gazebo/urdf/irb1200_ros2control.xacro (robot description, xacro)
@@ -153,29 +153,22 @@
     <gazebo reference="${prefix}base_link">
       <selfCollide>false</selfCollide>
-      <material>Gazebo/Orange</material>
     </gazebo>
     <gazebo reference="${prefix}link_1">
       <selfCollide>false</selfCollide>
-      <material>Gazebo/Orange</material>
     </gazebo>
     <gazebo reference="${prefix}link_2">
       <selfCollide>false</selfCollide>
-      <material>Gazebo/Orange</material>
     </gazebo>
     <gazebo reference="${prefix}link_3">
       <selfCollide>false</selfCollide>
-      <material>Gazebo/Orange</material>
     </gazebo>
     <gazebo reference="${prefix}link_4">
       <selfCollide>false</selfCollide>
-      <material>Gazebo/Orange</material>
     </gazebo>
     <gazebo reference="${prefix}link_5">
       <selfCollide>false</selfCollide>
-      <material>Gazebo/Orange</material>
     </gazebo>
     <gazebo reference="${prefix}link_6">
       <selfCollide>false</selfCollide>
-      <material>Gazebo/Orange</material>
     </gazebo>
     <gazebo reference="end_effector_frame_fixed_joint">

File: new_arm_ws/install/irb120_ros2_gazebo/share/irb120_ros2_gazebo/urdf/irb120_macro.urdf.xacro (robot description, xacro)
@@ -77,5 +77,5 @@
         <origin xyz="0 0 0" rpy="0 0 0"/>
         <geometry>
-          <mesh filename="file://$(find irb120_ros2_gazebo)/meshes/visual/base_link.stl"/>
+          <mesh filename="file://$(find irb120_ros2_gazebo)/meshes/visual/base_link.dae"/>
         </geometry>
         <xacro:material_abb_orange />
@@ -99,5 +99,5 @@
         <origin xyz="0 0 0" rpy="0 0 0"/>
         <geometry>
-          <mesh filename="file://$(find irb120_ros2_gazebo)/meshes/visual/link_1.stl"/>
+          <mesh filename="file://$(find irb120_ros2_gazebo)/meshes/visual/link_1.dae"/>
         </geometry>
         <xacro:material_abb_orange />
@@ -121,5 +121,5 @@
         <origin xyz="0 0 0" rpy="0 0 0"/>
         <geometry>
-          <mesh filename="file://$(find irb120_ros2_gazebo)/meshes/visual/link_2.stl"/>
+          <mesh filename="file://$(find irb120_ros2_gazebo)/meshes/visual/link_2.dae"/>
         </geometry>
         <xacro:material_abb_orange />
@@ -143,5 +143,5 @@
         <origin xyz="0 0 0" rpy="0 0 0"/>
         <geometry>
-          <mesh filename="file://$(find irb120_ros2_gazebo)/meshes/visual/link_3.stl"/>
+          <mesh filename="file://$(find irb120_ros2_gazebo)/meshes/visual/link_3.dae"/>
         </geometry>
         <xacro:material_abb_orange />
@@ -165,5 +165,5 @@
         <origin xyz="0 0 0" rpy="0 0 0"/>
         <geometry>
-          <mesh filename="file://$(find irb120_ros2_gazebo)/meshes/visual/link_4.stl"/>
+          <mesh filename="file://$(find irb120_ros2_gazebo)/meshes/visual/link_4.dae"/>
         </geometry>
         <xacro:material_abb_orange />
@@ -187,5 +187,5 @@
         <origin xyz="0 0 0" rpy="0 0 0"/>
         <geometry>
-          <mesh filename="file://$(find irb120_ros2_gazebo)/meshes/visual/link_5.stl"/>
+          <mesh filename="file://$(find irb120_ros2_gazebo)/meshes/visual/link_5.dae"/>
         </geometry>
         <xacro:material_abb_orange />
@@ -209,5 +209,5 @@
         <origin xyz="0 0 0" rpy="0 0 0"/>
         <geometry>
-          <mesh filename="file://$(find irb120_ros2_gazebo)/meshes/visual/link_6.stl"/>
+          <mesh filename="file://$(find irb120_ros2_gazebo)/meshes/visual/link_6.dae"/>
         </geometry>
         <xacro:material_abb_black />
@@ -230,5 +230,5 @@
       <limit effort="0" lower="-2.87979" upper="2.87979" velocity="4.36332"/>
       <axis xyz="0 0 1"/>
-      <dynamics damping="0.0" friction="0.0"/>
+      <dynamics damping="50.0" friction="1.0"/>
     </joint>
     <!-- joint_2 -->
@@ -239,5 +239,5 @@
       <limit effort="0" lower="-1.91986" upper="1.91986" velocity="4.36332"/>
       <axis xyz="0 1 0"/>
-      <dynamics damping="0.0" friction="0.0"/>
+      <dynamics damping="50.0" friction="1.0"/>
     </joint>
     <!-- joint_3 -->
@@ -248,5 +248,5 @@
       <limit effort="0" lower="-1.91986" upper="1.22173" velocity="4.36332"/>
       <axis xyz="0 1 0"/>
-      <dynamics damping="0.0" friction="0.0"/>
+      <dynamics damping="10.0" friction="1.0"/>
     </joint>
     <!-- joint_4 -->
@@ -257,5 +257,5 @@
       <limit effort="0" lower="-2.79253" upper="2.79253" velocity="5.58505"/>
       <axis xyz="1 0 0"/>
-      <dynamics damping="0.0" friction="0.0"/>
+      <dynamics damping="5.0" friction="1.0"/>
     </joint>
     <!-- joint_5 -->
@@ -266,5 +266,5 @@
       <limit effort="0" lower="-2.094395" upper="2.094395" velocity="5.58505"/>
       <axis xyz="0 1 0"/>
-      <dynamics damping="0.0" friction="0.0"/>
+      <dynamics damping="2.0" friction="1.0"/>
     </joint>
     <!-- joint_6 -->
@@ -275,5 +275,5 @@
       <limit effort="0" lower="-6.98132" upper="6.98132" velocity="7.33038"/>
       <axis xyz="1 0 0"/>
-      <dynamics damping="0.0" friction="0.0"/>
+      <dynamics damping="1.0" friction="1.0"/>
     </joint>
     <!-- end of joint list -->
@@ -307,10 +307,10 @@
         <visual>
           <geometry>
-            <mesh filename="file://$(find irb120_ros2_gazebo)/meshes/egp64/Schunk Gripper - ADAPTER.dae" />
-          </geometry>
-        </visual>
-        <collision>
-          <geometry>
-            <mesh filename="file://$(find irb120_ros2_gazebo)/meshes/egp64/Schunk Gripper - ADAPTER.dae" />
+            <mesh filename="file://$(find irb120_ros2_gazebo)/meshes/egp64/egp64_Adapter.dae" />
+          </geometry>
+        </visual>
+        <collision>
+          <geometry>
+            <mesh filename="file://$(find irb120_ros2_gazebo)/meshes/egp64/egp64_Adapter.dae" />
           </geometry>
         </collision>
@@ -340,5 +340,5 @@
         <visual>
           <geometry>
-            <mesh filename="file://$(find irb120_ros2_gazebo)/meshes/egp64/Schunk Gripper - BASE noAdapter.dae" />
+            <mesh filename="file://$(find irb120_ros2_gazebo)/meshes/egp64/egp64_BaseNoAdapter.dae" />
           </geometry>
           <material name="blue">
@@ -348,5 +348,5 @@
         <collision>
           <geometry>
-            <mesh filename="file://$(find irb120_ros2_gazebo)/meshes/egp64/Schunk Gripper - BASE noAdapter.dae" />
+            <mesh filename="file://$(find irb120_ros2_gazebo)/meshes/egp64/egp64_BaseNoAdapter.dae" />
           </geometry>
           <material name="blue"/>
@@ -367,5 +367,5 @@
         <visual>
           <geometry>
-            <mesh filename="file://$(find irb120_ros2_gazebo)/meshes/egp64/Schunk Gripper - LEFT FINGER BASE.dae" />
+            <mesh filename="file://$(find irb120_ros2_gazebo)/meshes/egp64/egp64_LeftFingerBase.dae" />
           </geometry>
           <material name="black">
@@ -375,5 +375,5 @@
         <collision>
           <geometry>
-            <mesh filename="file://$(find irb120_ros2_gazebo)/meshes/egp64/Schunk Gripper - LEFT FINGER BASE.dae" />
+            <mesh filename="file://$(find irb120_ros2_gazebo)/meshes/egp64/egp64_LeftFingerBase.dae" />
           </geometry>
           <material name="black" />
@@ -386,4 +386,5 @@
         <origin xyz="0.01483 -0.00782 0" rpy="0 0 0" />
         <axis xyz="-1 0 0" />
+        <dynamics damping="1.0" friction="1.0"/>
       </joint>
       <!-- LEFT FINGERTIP -->
@@ -396,5 +397,5 @@
         <visual>
           <geometry>
-            <mesh filename="file://$(find irb120_ros2_gazebo)/meshes/egp64/Schunk Gripper - LEFT FINGER.dae" />
+            <mesh filename="file://$(find irb120_ros2_gazebo)/meshes/egp64/egp64_LeftFinger.dae" />
           </geometry>
           <material name="silver">
@@ -404,5 +405,5 @@
         <collision>
           <geometry>
-            <mesh filename="file://$(find irb120_ros2_gazebo)/meshes/egp64/Schunk Gripper - LEFT FINGER.dae" />
+            <mesh filename="file://$(find irb120_ros2_gazebo)/meshes/egp64/egp64_LeftFinger.dae" />
           </geometry>
           <material name="black"/>
@@ -423,5 +424,5 @@
         <visual>
           <geometry>
-            <mesh filename="file://$(find irb120_ros2_gazebo)/meshes/egp64/Schunk Gripper - RIGHT FINGER BASE.dae" />
+            <mesh filename="file://$(find irb120_ros2_gazebo)/meshes/egp64/egp64_RightFingerBase.dae" />
           </geometry>
           <material name="black"/>
@@ -429,5 +430,5 @@
         <collision>
           <geometry>
-            <mesh filename="file://$(find irb120_ros2_gazebo)/meshes/egp64/Schunk Gripper - RIGHT FINGER BASE.dae" />
+            <mesh filename="file://$(find irb120_ros2_gazebo)/meshes/egp64/egp64_RightFingerBase.dae" />
           </geometry>
           <material name="black"/>
@@ -440,4 +441,5 @@
         <origin xyz="-0.0153 -0.00602 0" rpy="0 0 0" />
         <axis xyz="1 0 0" />
+        <dynamics damping="1.0" friction="1.0"/>
       </joint>
       <!-- RIGHT FINGERTIP -->
@@ -450,5 +452,5 @@
         <visual>
           <geometry>
-            <mesh filename="file://$(find irb120_ros2_gazebo)/meshes/egp64/Schunk Gripper - RIGHT FINGER.dae" />
+            <mesh filename="file://$(find irb120_ros2_gazebo)/meshes/egp64/egp64_RightFinger.dae" />
           </geometry>
           <material name="silver" />
@@ -456,5 +458,5 @@
         <collision>
           <geometry>
-            <mesh filename="file://$(find irb120_ros2_gazebo)/meshes/egp64/Schunk Gripper - RIGHT FINGER.dae" />
+            <mesh filename="file://$(find irb120_ros2_gazebo)/meshes/egp64/egp64_RightFinger.dae" />
           </geometry>
           <material name="black"/>
@@ -485,4 +487,5 @@
         <axis xyz="1 0 0" />
         <origin xyz="0.033 -0.018 0.15" rpy="0 0 0"/>
+        <dynamics damping="1.0" friction="1.0"/>
       </joint>
     </xacro:if>

File: new_arm_ws/install/irb120_ros2_gazebo/share/irb120_ros2_gazebo/urdf/irb120_ros2control.xacro (robot description, xacro)
@@ -208,29 +208,22 @@
     <gazebo reference="${prefix}base_link">
       <selfCollide>false</selfCollide>
-      <material>Gazebo/Orange</material>
     </gazebo>
     <gazebo reference="${prefix}link_1">
       <selfCollide>false</selfCollide>
-      <material>Gazebo/Orange</material>
     </gazebo>
     <gazebo reference="${prefix}link_2">
       <selfCollide>false</selfCollide>
-      <material>Gazebo/Orange</material>
     </gazebo>
     <gazebo reference="${prefix}link_3">
       <selfCollide>false</selfCollide>
-      <material>Gazebo/Orange</material>
     </gazebo>
     <gazebo reference="${prefix}link_4">
       <selfCollide>false</selfCollide>
-      <material>Gazebo/Orange</material>
     </gazebo>
     <gazebo reference="${prefix}link_5">
       <selfCollide>false</selfCollide>
-      <material>Gazebo/Orange</material>
     </gazebo>
     <gazebo reference="${prefix}link_6">
       <selfCollide>false</selfCollide>
-      <material>Gazebo/Orange</material>
     </gazebo>
     <!-- =================================== -->

File: new_arm_ws/install/irb6640_ros2_gazebo/share/irb6640_ros2_gazebo/urdf/irb6640_macro.urdf.xacro (robot description, xacro)
@@ -265,5 +265,5 @@
       <child link="${prefix}link_1"/>
       <limit effort="0" lower="-2.967" upper="2.967" velocity="1.7453"/>
-      <dynamics damping="0.0" friction="0.0"/>
+      <dynamics damping="50.0" friction="1.0"/>
     </joint>
     <!-- joint_2 -->
@@ -274,5 +274,5 @@
       <child link="${prefix}link_2"/>
       <limit effort="0" lower="-1.134" upper="1.4855" velocity="1.5707"/>
-      <dynamics damping="0.0" friction="0.0"/>
+      <dynamics damping="50.0" friction="1.0"/>
     </joint>
     <!-- joint_3 -->
@@ -283,5 +283,5 @@
       <child link="${prefix}link_3"/>
       <limit effort="0" lower="-3.142" upper="1.222" velocity="1.5707"/>
-      <dynamics damping="0.0" friction="0.0"/>
+      <dynamics damping="10.0" friction="1.0"/>
     </joint>
     <!-- joint_4 -->
@@ -292,5 +292,5 @@
       <child link="${prefix}link_4"/>
       <limit effort="0" lower="-5.236" upper="5.236" velocity="2.9671"/>
-      <dynamics damping="0.0" friction="0.0"/>
+      <dynamics damping="5.0" friction="1.0"/>
     </joint>
     <!-- joint_5 -->
@@ -301,4 +301,5 @@
       <child link="${prefix}link_5"/>
       <limit effort="0" lower="-2.094" upper="2.094" velocity="2.4435"/>
+      <dynamics damping="2.0" friction="1.0"/>
     </joint>
     <!-- joint_6 -->
@@ -309,5 +310,5 @@
       <child link="${prefix}link_6"/>
       <limit effort="0" lower="-6.283" upper="6.283" velocity="3.3161"/>
-      <dynamics damping="0.0" friction="0.0"/>
+      <dynamics damping="1.0" friction="1.0"/>
     </joint>
     <!-- end of joint list -->
@@ -326,5 +327,5 @@
       <child link="${prefix}link_cylinder"/>
       <mimic joint="${prefix}joint_2" multiplier="-0.25"/>
-      <dynamics damping="0.0" friction="0.0"/>
+      <dynamics damping="10.0" friction="1.0"/>
     </joint>
     <!-- piston joint

File: new_arm_ws/install/panda_ros2_gazebo/share/panda_ros2_gazebo/urdf/panda_macro.urdf.xacro (robot description, xacro)
@@ -114,4 +114,5 @@
       <axis xyz="0 0 1"/>
       <limit effort="87" lower="-2.8973" upper="2.8973" velocity="2.1750"/>
+      <dynamics damping="50.0" friction="1.0"/>
     </joint>
     <!-- panda_link2 -->
@@ -145,4 +146,5 @@
       <axis xyz="0 0 1"/>
       <limit effort="87" lower="-1.7628" upper="1.7628" velocity="2.1750"/>
+      <dynamics damping="50.0" friction="1.0"/>
     </joint>
     <!-- panda_link3 -->
@@ -176,4 +178,5 @@
       <axis xyz="0 0 1"/>
       <limit effort="87" lower="-2.8973" upper="2.8973" velocity="2.1750"/>
+      <dynamics damping="10.0" friction="1.0"/>
     </joint>
     <!-- panda_link4-->
@@ -208,4 +211,5 @@
       <limit effort="87" lower="-3.0718" upper="0.0698" velocity="2.1750"/>
       <!-- upper should be -0.0698, but that brakes simulation when initial position for this joint is 0.0 -->
+      <dynamics damping="10.0" friction="1.0"/>
     </joint>
     <!-- panda_link5 -->
@@ -239,4 +243,5 @@
       <axis xyz="0 0 1"/>
       <limit effort="12" lower="-2.8973" upper="2.8973" velocity="2.6100"/>
+      <dynamics damping="5.0" friction="1.0"/>
     </joint>
     <!-- panda_link6 -->
@@ -270,4 +275,5 @@
       <axis xyz="0 0 1"/>
       <limit effort="12" lower="-0.0175" upper="3.7525" velocity="2.6100"/>
+      <dynamics damping="5.0" friction="1.0"/>
     </joint>
     <!-- panda_link7 -->
@@ -301,4 +307,5 @@
       <axis xyz="0 0 1"/>
       <limit effort="12" lower="-3.15" upper="3.15" velocity="2.6100"/>
+      <dynamics damping="1.0" friction="1.0"/>
     </joint>
     <!-- panda_link8 -->
@@ -391,4 +398,5 @@
       <axis xyz="0 1 0"/>
       <limit effort="20" lower="-0.001" upper="0.04" velocity="0.3"/>
+      <dynamics damping="1.0" friction="1.0"/>
     </joint>
     <joint name="panda_finger_joint2" type="prismatic">
@@ -398,4 +406,5 @@
       <axis xyz="0 -1 0"/>
       <limit effort="20" lower="-0.001" upper="0.04" velocity="0.3"/>
+      <dynamics damping="1.0" friction="1.0"/>
     </joint>
     <!-- End-Effector frame -->

File: new_arm_ws/install/panda_ros2_gazebo/share/panda_ros2_gazebo/urdf/panda_ros2control.xacro (robot description, xacro)
@@ -201,49 +201,37 @@
     <gazebo reference="panda_link0">
       <selfCollide>false</selfCollide>
-      <material>Gazebo/Orange</material>
     </gazebo>
     <gazebo reference="panda_link1">
       <selfCollide>false</selfCollide>
-      <material>Gazebo/Orange</material>
     </gazebo>
     <gazebo reference="panda_link2">
       <selfCollide>false</selfCollide>
-      <material>Gazebo/Orange</material>
     </gazebo>
     <gazebo reference="panda_link3">
       <selfCollide>false</selfCollide>
-      <material>Gazebo/Orange</material>
     </gazebo>
     <gazebo reference="panda_link4">
       <selfCollide>false</selfCollide>
-      <material>Gazebo/Orange</material>
     </gazebo>
     <gazebo reference="panda_link5">
       <selfCollide>false</selfCollide>
-      <material>Gazebo/Orange</material>
     </gazebo>
     <gazebo reference="panda_link6">
       <selfCollide>false</selfCollide>
-      <material>Gazebo/Orange</material>
     </gazebo>
     <gazebo reference="panda_link7">
       <selfCollide>false</selfCollide>
-      <material>Gazebo/Orange</material>
     </gazebo>
     <gazebo reference="panda_link8">
       <selfCollide>false</selfCollide>
-      <material>Gazebo/Orange</material>
     </gazebo>
     <gazebo reference="panda_hand">
       <selfCollide>false</selfCollide>
-      <material>Gazebo/Orange</material>
     </gazebo>
     <gazebo reference="panda_leftfinger">
       <selfCollide>false</selfCollide>
-      <material>Gazebo/Orange</material>
     </gazebo>
     <gazebo reference="panda_rightfinger">
       <selfCollide>false</selfCollide>
-      <material>Gazebo/Orange</material>
     </gazebo>
     <gazebo reference="end_effector_frame_fixed_joint">
