Commit message: Mais testes a caminho

File: pfc_ws/install/testing/share/testing/urdf/pfcbot.xacro (robot description, xacro)
@@ -7,4 +7,22 @@
   <!--xacro:include filename="$(find testing)/urdf/materials.xacro" /-->
   <xacro:manipulator namespace=""/>
+  <link name="dummy_root_link">
+    <inertial>
+      <mass value="0.0"/> <!-- No mass -->
+      <origin xyz="0 0 0"/> <!-- Centered -->
+      <inertia ixx="0.0" ixy="0.0" ixz="0.0" iyy="0.0" iyz="0.0" izz="0.0"/> <!-- No inertia -->
+    </inertial>
+    <visual>
+      <geometry>
+        <sphere radius="0.0001"/> <!-- Invisible -->
+      </geometry>
+    </visual>
+  </link>
+  <!-- Joint to connect Dummy Link to the Base of the Robot -->
+  <joint name="dummy_to_body_joint" type="fixed">
+    <origin xyz="0 0 0" rpy="0 0 0"/>
+    <parent link="dummy_root_link"/> <!-- Parent is the dummy link -->
+    <child link="body_link"/> <!-- Child is the body link -->
+  </joint>
   <!-- This is the body of the robot -->
   <link name="body_link">

Commit message: Muitas e muitas tentativas de fazer dar certo

File: pfc_ws/install/testing/share/testing/urdf/pfcbot.xacro (robot description, xacro)
@@ -8,14 +8,19 @@
   <xacro:manipulator namespace=""/>
   <link name="dummy_root_link">
-    <inertial>
-      <mass value="0.0"/> <!-- No mass -->
-      <origin xyz="0 0 0"/> <!-- Centered -->
-      <inertia ixx="0.0" ixy="0.0" ixz="0.0" iyy="0.0" iyz="0.0" izz="0.0"/> <!-- No inertia -->
-    </inertial>
-    <visual>
-      <geometry>
-        <sphere radius="0.0001"/> <!-- Invisible -->
-      </geometry>
-    </visual>
+    <!--inertial>
+      <mass value="0.0"/>
+      <origin xyz="0 0 0"/>
+      <inertia ixx="0.0" ixy="0.0" ixz="0.0" iyy="0.0" iyz="0.0" izz="0.0"/>
+    </inertial-->
+    <visual>
+      <geometry>
+        <sphere radius="0.0001"/>
+      </geometry>
+    </visual>
+    <collision>
+      <geometry>
+        <sphere radius="0.0001"/>
+      </geometry>
+    </collision>
   </link>
   <!-- Joint to connect Dummy Link to the Base of the Robot -->

Commit message: Updates

File: pfc_ws/install/testing/share/testing/urdf/pfcbot.xacro (robot description, xacro)
@@ -7,27 +7,26 @@
   <!--xacro:include filename="$(find testing)/urdf/materials.xacro" /-->
   <xacro:manipulator namespace=""/>
-  <link name="dummy_root_link">
-    <!--inertial>
-      <mass value="0.0"/>
-      <origin xyz="0 0 0"/>
-      <inertia ixx="0.0" ixy="0.0" ixz="0.0" iyy="0.0" iyz="0.0" izz="0.0"/>
-    </inertial-->
-    <visual>
-      <geometry>
-        <sphere radius="0.0001"/>
-      </geometry>
-    </visual>
-    <collision>
-      <geometry>
-        <sphere radius="0.0001"/>
-      </geometry>
-    </collision>
-  </link>
-  <!-- Joint to connect Dummy Link to the Base of the Robot -->
-  <joint name="dummy_to_body_joint" type="fixed">
-    <origin xyz="0 0 0" rpy="0 0 0"/>
-    <parent link="dummy_root_link"/> <!-- Parent is the dummy link -->
-    <child link="body_link"/> <!-- Child is the body link -->
-  </joint>
+  <link name="world">
+    <visual>
+        <origin xyz="0 0 0" rpy="0 0 0"/>
+        <geometry>
+            <box size="5.0 5.0 0.05"/>
+        </geometry>
+        <material name="Grey">
+            <color rgba="0.7 0.7 0.7 1.0"/>
+        </material>
+    </visual>
+    <collision>
+        <origin xyz="0 0 0" rpy="0 0 0"/>
+        <geometry>
+            <box size="5.0 5.0 0.05"/>
+        </geometry>
+    </collision>
+  </link>
+    <joint name="worldy_joint" type="fixed">
+        <origin xyz="0 0 0.0025" rpy="0 0 0"/>
+        <parent link="world"/>
+        <child link="body_link"/>
+    </joint>
   <!-- This is the body of the robot -->
   <link name="body_link">
