Commit message: Pick Script

File: new_arm_ws/src/ros2_RobotSimulation/ros2_grasping/urdf/box.urdf (robot description, URDF)
Before this commit: robot box, 1 links, 0 joints
Links:
- link box: geometry collision box size=0.04 0.06 0.04; visual box size=0.04 0.06 0.04

Commit message: Pick and Place completamente funcional

File: new_arm_ws/src/ros2_RobotSimulation/ros2_grasping/urdf/box.urdf (robot description, URDF)
Before this commit: robot box, 1 links, 0 joints
Links:
- link box: geometry collision box size=0.05 0.03 0.08; visual box size=0.05 0.03 0.08
