Commit message: Levantei bandeira branca

File: new_arm_ws/src/ros2_RobotSimulation/ABBRobots/IRB120/irb120_ros2_gazebo/urdf/irbTEST.urdf.xacro (robot description, xacro)
@@ -52,8 +52,8 @@
   <xacro:arg name="cell_layout_1" default="false"/>
   <xacro:property name="cell_layout_1" value="$(arg cell_layout_1)"/>
-  <xacro:arg name="cell_layout_2" default="false"/>
+  <!--xacro:arg name="cell_layout_2" default="false"/>
   <xacro:property name="cell_layout_2" value="$(arg cell_layout_2)"/>
   <xacro:arg name="cell_layout_3" default="false"/>
-  <xacro:property name="cell_layout_3" value="$(arg cell_layout_3)"/>
+  <xacro:property name="cell_layout_3" value="$(arg cell_layout_3)"/-->
   <!-- END-EFFECTOR:  -->
   <xacro:arg name="EE_no" default="false"/>
@@ -69,5 +69,5 @@
   />
   <!-- Gazebo WORLD link: -->
-  <link name="world"/>
+  <!--link name="world"/-->
   <!-- ========== ========== ========== ========== ========== ========== -->
   <!-- CELL LAYOUT SELECTION: -->
@@ -80,5 +80,5 @@
   </xacro:if>
   <!-- CELL LAYOUT N2) ABB IRB120 Robot in Cranfield University cell: -->
-  <xacro:if value="${cell_layout_2}">
+  <!--xacro:if value="${cell_layout_2}">
     <link name="cell">
       <visual>
@@ -108,7 +108,7 @@
       <origin xyz="0.0 0.0 0.015" rpy="0.0 0.0 0.0" />
     </joint>
-  </xacro:if>
+  </xacro:if-->
   <!-- CELL LAYOUT N3) ABB IRB120 + PICK & PLACE layout: -->
-  <xacro:if value="${cell_layout_3}">
+  <!--xacro:if value="${cell_layout_3}">
     <link name='irb120_block'>
       <inertial>
@@ -170,4 +170,4 @@
       <origin xyz="0.7 0.0 0.35" rpy="0.0 0.0 0.0" />
     </joint>
-  </xacro:if>
+  </xacro:if-->
 </robot>

File: new_arm_ws/src/ros2_RobotSimulation/ABBRobots/IRB120/irb120_ros2_gazebo/urdf/test/irbTESTmacro.urdf.xacro (robot description, xacro)
@@ -124,5 +124,5 @@
       </inertial>
       <visual>
-        <origin xyz="0 0 0.45" rpy="0 0 0"/>
+        <origin xyz="0 0 0.2" rpy="0 0 0"/>
         <geometry>
           <mesh filename="file://$(find irb120_ros2_gazebo)/meshes/visual/base_link.dae"/>
@@ -131,5 +131,5 @@
       </visual>
       <collision>
-        <origin xyz="0 0 0.45" rpy="0 0 0"/>
+        <origin xyz="0 0 0.2" rpy="0 0 0"/>
         <geometry>
           <mesh filename="file://$(find irb120_ros2_gazebo)/meshes/collision/base_link.stl"/>
@@ -139,5 +139,5 @@
     </link>
     <joint name="manipulator_fixed" type="fixed">
-        <origin xyz="0 0 0.45" rpy="0 0 0"/>
+        <origin xyz="0 0 0.2" rpy="0 0 0"/>
         <parent link="body_link"/>
         <child link="base_link"/>
